File: PowerExtender_x2.kicad_pcb (KiCad board)
At the start: 2 copper layers, 82.8 x 21.4 mm, 10 parts, among them J1 Conn_01x05, J2 Conn_01x05, J3 Conn_01x05, J4 Conn_01x05, J6 Conn_01x05, J7 Conn_01x05

Commit message: Label change from "VIN module" to "PnP Power Module"
Parts:
- renumbered J6 to J5, J7 to J6
Connections:
- J1 pad 3: (no net) -> unconnected-(J1-Pin_3-Pad3)
- J2 pad 3: (no net) -> unconnected-(J2-Pin_3-Pad3)_1
- J3 pad 3: (no net) -> unconnected-(J3-Pin_3-Pad3)_1
- J4 pad 3: (no net) -> unconnected-(J4-Pin_3-Pad3)_1
- J5 pad 3: (no net) -> unconnected-(J5-Pin_3-Pad3)_1
- J6 pad 3: (no net) -> unconnected-(J6-Pin_3-Pad3)
Other:
- board text added: "PnP Power Module"
- board text removed: "VIN module"
