File: panel.kicad_pcb (KiCad board)
At the start: 2 copper layers, 96.8 x 78.2 mm, 42 parts, among them J1 Conn_01x05, J2 Conn_01x05, J3 Conn_01x05, J4 Conn_01x05, J6 Conn_01x05, J7 Conn_01x05

Commit message: Label change from "VIN module" to "PnP Power Module"
Parts:
- removed the J6 at (166.0, 59.1)
- removed the J6 at (166.0, 80.5)
- removed the J6 at (166.0, 37.7)
- removed J7 (x3): Conn_01x05, PnP_Library:PinSocket_1x05_P2.54mm_Vertical_SMD_Pin1Left
- added J5: Conn_01x05, PnP_Library:PinSocket_1x05_P2.54mm_Vertical_SMD_Pin1Right, F.Cu at (166.0, 37.7)
- added J5: Conn_01x05, PnP_Library:PinSocket_1x05_P2.54mm_Vertical_SMD_Pin1Right, F.Cu at (166.0, 59.1)
- added J5: Conn_01x05, PnP_Library:PinSocket_1x05_P2.54mm_Vertical_SMD_Pin1Right, F.Cu at (166.0, 80.5)
- added J6: Conn_01x05, PnP_Library:PinSocket_1x05_P2.54mm_Vertical_SMD_Pin1Left, F.Cu at (186.0, 59.1)
- added J6: Conn_01x05, PnP_Library:PinSocket_1x05_P2.54mm_Vertical_SMD_Pin1Left, F.Cu at (186.0, 37.7)
- added J6: Conn_01x05, PnP_Library:PinSocket_1x05_P2.54mm_Vertical_SMD_Pin1Left, F.Cu at (186.0, 80.5)
Connections:
- J1 pad 3: (no net) -> Board_0-unconnected-(J1-Pin_3-Pad3)
- J1 pad 3: (no net) -> Board_2-unconnected-(J1-Pin_3-Pad3)
- J1 pad 3: (no net) -> Board_1-unconnected-(J1-Pin_3-Pad3)
- J2 pad 3: (no net) -> Board_0-unconnected-(J2-Pin_3-Pad3)_1
- J2 pad 3: (no net) -> Board_2-unconnected-(J2-Pin_3-Pad3)_1
- J2 pad 3: (no net) -> Board_1-unconnected-(J2-Pin_3-Pad3)_1
- J3 pad 3: (no net) -> Board_0-unconnected-(J3-Pin_3-Pad3)_1
- J3 pad 3: (no net) -> Board_2-unconnected-(J3-Pin_3-Pad3)_1
- J3 pad 3: (no net) -> Board_1-unconnected-(J3-Pin_3-Pad3)_1
- J4 pad 3: (no net) -> Board_1-unconnected-(J4-Pin_3-Pad3)_1
- J4 pad 3: (no net) -> Board_2-unconnected-(J4-Pin_3-Pad3)_1
- J4 pad 3: (no net) -> Board_0-unconnected-(J4-Pin_3-Pad3)_1
Other:
- board text added: "PnP Power Module"
- board text removed: "VIN module"
